File: Esp32InfraredController/Esp32InfraredController.kicad_pcb (KiCad board)
At the start: 2 copper layers, 27.8 x 41.2 mm, 6 parts, among them J1 Conn_02x05_Odd_Even, Q1 SS8050, U1 ESP32-C3_SUPERMINI_SMD

Commit message: no message
Parts:
- added J2: Conn_01x02_Pin, Connector_PinHeader_1.00mm:PinHeader_1x02_P1.00mm_Vertical, F.Cu at (105.0, 64.0)
- J1: moved to B.Cu
- moved Q1 9.55 mm to (115.5, 71.9), turned to 90 degrees
- moved U1 9.50 mm to (117.5, 57.9)
- moved R2 9.01 mm to (112.5, 72.3)
- moved R1 8.86 mm to (118.5, 72.3)
- moved D1 2.51 mm to (115.7, 84.0)
Connections:
- J1 pad 10: /GPIO4 -> /GPIO7
- J1 pad 3: /GPIO5 -> /GPIO4
- J1 pad 4: /GPIO6 -> /GPIO3
- J1 pad 5: /GPIO7 -> /GPIO2
- J1 pad 6: /GPIO8 -> /GPIO1
- J1 pad 7: /GPIO1 -> /GPIO6
- J1 pad 8: /GPIO2 -> /GPIO8
- J1 pad 9: /GPIO3 -> /GPIO5
- U1 pad 20: unconnected-(U1-GPIO20-Pad20) -> Net-(J2-Pin_2)
- U1 pad 21: unconnected-(U1-GPIO21-Pad21) -> Net-(J2-Pin_1)
Routing:
- net GNDREF: track 57.2 -> 31.4 mm, vias 0 -> 3
- net /3.3V: track 49.7 -> 24.7 mm, vias 0 -> 3
- net /GPIO7: track 20.3 -> 3.30 mm, vias 2 -> 1
- net /GPIO3: track 24.3 -> 10.4 mm, vias 2 -> 1
- net /GPIO1: track 30.3 -> 16.4 mm, vias 2 -> 1
- net /GPIO5: track 14.2 -> 3.28 mm, vias 2 -> 1
- net /GPIO8: track 17.7 -> 8.38 mm, vias 2 -> 1
- net Net-(D1-K): track 4.64 -> 13.1 mm
- net Net-(D1-A): track 2.52 -> 10.9 mm
- net Net-(J2-Pin_1): track 0.00 -> 5.25 mm
- net Net-(J2-Pin_2): track 0.00 -> 4.61 mm
- net /GPIO6: track 11.7 -> 7.05 mm, vias 2 -> 1
- net /GPIO4: track 16.5 -> 12.9 mm, vias 2 -> 1
- net /GPIO2: track 22.3 -> 18.9 mm, vias 2 -> 1
- net Net-(Q1-B): track 4.31 -> 2.16 mm
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
Commit message: no message
Parts:
- added J3: Conn_01x04_Pin, Connector_PinHeader_1.00mm:PinHeader_1x04_P1.00mm_Vertical, F.Cu at (130.0, 61.0)
Connections:
- J1 pad 6: /GPIO1 -> /GPIO9
- U1 pad 0: unconnected-(U1-GPIO0-Pad0) -> /GPIO0
- U1 pad 9: unconnected-(U1-GPIO9-Pad9) -> /GPIO9
Routing:
- net /GPIO9: track 0.00 -> 12.0 mm, vias 0 -> 1
- net /GPIO1: track 16.4 -> 4.95 mm
- net GNDREF: track 31.4 -> 42.9 mm
- net /3.3V: track 24.7 -> 34.6 mm
- net /GPIO0: track 0.00 -> 5.25 mm, vias 0 -> 1
- net /GPIO4: track 12.9 -> 12.3 mm
- net /GPIO3: track 10.4 -> 9.79 mm
- net /GPIO2: track 18.9 -> 18.3 mm
- net Net-(J2-Pin_2): track 4.61 -> 4.95 mm, vias 0 -> 1
- net Net-(J2-Pin_1): vias 0 -> 1
Other:
- board text added: "G"
- board text added: "P0"
- board text added: "P1"
- board text added: "RX"
- board text added: "TX"
- board text added: "V"

Commit message: .
Parts:
- J2: footprint Connector_PinHeader_1.00mm:PinHeader_1x02_P1.00mm_Vertical -> Connector_PinHeader_2.54mm:PinHeader_1x02_P2.54mm_Vertical
- J3: footprint Connector_PinHeader_1.00mm:PinHeader_1x04_P1.00mm_Vertical -> Connector_PinHeader_2.54mm:PinHeader_1x04_P2.54mm_Vertical
- moved J3 3.12 mm to (129.2, 58.0)
- moved J2 1.78 mm to (105.6, 65.7)
Routing:
- net /GPIO0: track 5.25 -> 3.79 mm
- net GNDREF: track 42.9 -> 41.6 mm
- net /GPIO1: track 4.95 -> 4.13 mm
- net /3.3V: track 34.6 -> 35.5 mm
- net Net-(J2-Pin_2): track 4.95 -> 4.30 mm
Other:
- board text removed: "G"
- board text removed: "P0"
- board text removed: "P1"
- board text removed: "RX"
- board text removed: "TX"
- board text removed: "V"

Commit message: no message
Other:
- board text added: "Liebeskind 2025.03.07"
